File: IR_UART.kicad_pcb (KiCad board)
At the start: 2 copper layers, 35 x 22 mm, 18 parts, among them J1 USB_C, Q1 AO3400A, Q2 AO3400A, Q3 AO3400A, Q4 IR_PHOTO, U1 CH340N

Commit message: MkI PCB Done
Parts:
- JP1, JP2: moved to B.Cu
- moved JP1 54.0 mm to (98.3, 81.2), turned to 180 degrees
- moved JP2 21.7 mm to (98.3, 85.8), turned to 180 degrees
- moved Q3 3.61 mm to (91.0, 90.6)
- moved R4 3.61 mm to (91.5, 88.0)
- moved R5 3.61 mm to (91.5, 86.4)
- moved C2 3.10 mm to (105.8, 88.8)
- moved C1 3.10 mm to (101.4, 88.8)
- moved U1 3.10 mm to (103.6, 83.5)
- moved R3 2.79 mm to (91.5, 75.5), turned to 0 degrees
- moved Q2 2.60 mm to (92.1, 78.1), turned to 0 degrees
- moved Q1 1.10 mm to (86.4, 75.5)
- moved R1 1.10 mm to (86.9, 79.7)
- moved R2 1.10 mm to (86.9, 78.1)
Routing:
- net /USB_5V: track 12.9 -> 40.7 mm, vias 2 -> 5
- net /IR_RX: track 0.00 -> 12.7 mm, vias 0 -> 1
- net /IR_TX: track 0.00 -> 11.3 mm, vias 0 -> 1
- net /RECV: track 17.0 -> 26.5 mm, vias 0 -> 1
- net /!RECV: track 9.75 -> 14.1 mm, vias 0 -> 1
- net /!SEND: track 17.9 -> 14.0 mm, vias 0 -> 1
- net /USB_D-: track 23.7 -> 26.8 mm
- net /USB_D+: track 26.0 -> 29.1 mm
- net Net-(D1-K): track 3.79 -> 2.69 mm
- net Net-(D1-A): track 8.66 -> 7.88 mm
- net /SEND: track 12.2 -> 12.8 mm, vias 0 -> 1
- net GND: vias 13 -> 7
Other:
- board text added: "INVERT"
- board text added: "NORMAL"
- board text added: "RECV"
- board text added: "SEND"
- board text added: "USB to IR UART Adapter MkI 24 Mar 2026"
